File: Onboarding/Onbaording/_autosave-Onbaording.kicad_pcb (KiCad board)
At the start: 2 copper layers, 85 x 20 mm, 3 parts, among them J1 Screw_Terminal_2x2.54

Commit message: made more progress
Parts:
- moved D1 102.1 mm to (196.1, 64.0), turned to 0 degrees
- moved R1 90.3 mm to (191.3, 60.0), turned to 0 degrees
- moved J1 84.9 mm to (189.9, 66.4)
Connections:
- net Net-(J1-Pin_2) renamed +3V3
Routing:
- net +3V3: track 10.2 -> 0.00 mm
- net Net-(D1-A): track 7.41 -> 0.00 mm
- net GND: track 2.00 -> 0.00 mm, vias 1 -> 0
Other:
- board size 85 x 20 mm -> 20 x 20 mm
