File: Onboarding/Onbaording/Onbaording.kicad_pcb (KiCad board)
At the start: 2 copper layers, 20 x 20 mm, 3 parts, among them J1 Screw_Terminal_2x2.54

Commit message: made more progress
Other:
- board size 20 x 20 mm -> 85 x 20 mm
Changed lines of the file:
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@@
 		(tags "resistor")
 		(property "Reference" "R1"
-			(at 0 -3 360)
+			(at 0 -3 0)
 			(layer "F.SilkS")
 			(effects
@@
 		)
 		(property "Value" "200R_2W"
-			(at 0 2.62 360)
+			(at 0 2.62 0)
 			(layer "F.Fab")
 			(effects
@@
 		)
 		(property "Footprint" "rsx_resistors:R_2512_6332Metric"
-			(at 0 0 360)
+			(at 0 0 0)
 			(layer "F.Fab")
 			(hide yes)
@@
 		)
 		(property "Datasheet" ""
-			(at 0 0 360)
+			(at 0 0 0)
 			(layer "F.Fab")
 			(hide yes)
@@
 		)
 		(property "Description" "RES SMD 200 OHM 1% 2W 2512"
-			(at 0 0 360)
+			(at 0 0 0)
 			(layer "F.Fab")
 			(hide yes)
@@
 		)
 		(fp_text user "${REFERENCE}"
-			(at 0 0 360)
+			(at 0 0 0)
 			(layer "F.Fab")
 			(effects
@@
 	)
 	(gr_line
+		(start 156 54)
+		(end 176 54)
+		(stroke
+			(width 0.05)
+			(type default)
+		)
+		(layer "Edge.Cuts")
+	)
+	(gr_line
 		(start 92 54)
 		(end 110 54)
@@
 	)
 	(gr_line
+		(start 176 54)
+		(end 176 74)
+		(stroke
+			(width 0.05)
+			(type default)
+		)
+		(layer "Edge.Cuts")
+	)
+	(gr_line
+		(start 156 74)
+		(end 156 54)
+		(stroke
+			(width 0.05)
+			(type default)
+		)
+		(layer "Edge.Cuts")
+	)
+	(gr_line
 		(start 111 55)
 		(end 111 73)
 		(stroke
 			(width 0.05)
+			(type default)
+		)
+		(layer "Edge.Cuts")
+	)
+	(gr_line
+		(start 176 74)
+		(end 156 74)
+		(stroke
+			(width 0.05)

Commit message: more stuff
Parts:
- moved R1 70.0 mm to (171.0, 60.0), turned to 90 degrees
- moved D1 67.3 mm to (161.0, 59.0), turned to 0 degrees
- moved J1 58.8 mm to (163.8, 67.0)
Connections:
- net Net-(J1-Pin_2) renamed +3V3
Routing:
- net +3V3: track 10.2 -> 0.00 mm
- net Net-(D1-A): track 7.41 -> 0.00 mm
- net GND: track 2.00 -> 0.00 mm, vias 1 -> 0
Other:
- board size 85 x 20 mm -> 20 x 20 mm
